File: brass_board/PCB/main_board/main_board.kicad_sch (KiCad schematic)
At the start: 94 parts

Commit message: Added Arduino
Parts:
- added A1: (no value), symbol MCU_Module:Arduino_Nano_v3.x
- added J13: (no value), symbol Connector:Conn_01x02_Male
- added Q2: 2N2219, Package_TO_SOT_THT:TO-39-3, symbol Transistor_BJT:2N2219
- added R44: (no value), symbol Device:R_Small_US
- added R45: R_Small_US, symbol Device:R_Small_US
Connections:
- net +5V: now also A1.30 (VIN), R45.1
- net GND: now also A1.29 (GND), A1.4 (GND), J13.2 (Pin_2), Q2.1 (E)
- net at U10.22 (15_A1_RX3_SPDIF_IN), U11.22 (15_A1_RX3_SPDIF_IN): now also R44.1
- new net: A1.5 (D2), Q2.3 (C), R45.2
- new net: A1.7 (D4), J13.1 (Pin_1)
- new net: Q2.2 (B), R44.2
Other:
- moved on the sheet: C3, C4, FB1, FB2, FB3, J10, J6, J8, J9, Q1, R16, R17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

Commit message: Added test points and line driver for laser trigger
Parts:
- added C10, C12, C13: C_Small, symbol Device:C_Small
- added C11: (no value), symbol Device:C_Small
- added J14: Conn_POS_input_A, Connector_PinHeader_2.54mm:PinHeader_1x03_P2.54mm_Vertical, symbol Connector:Conn_01x03_Male
- added J15: Conn_POS_input_B, Connector_PinHeader_2.54mm:PinHeader_1x03_P2.54mm_Vertical, symbol Connector:Conn_01x03_Male
- added J16, J17, J18: (no value), symbol Connector_Generic:Conn_02x02_Odd_Even
- added J19: Conn_ADC, symbol Connector:Conn_01x04_Male
- added J20: Conn_ADC, Connector_PinHeader_2.54mm:PinHeader_1x03_P2.54mm_Vertical, symbol Connector:Conn_01x03_Male
- added J21, J23, J24: Conn_02x02_Odd_Even, Connector_PinHeader_2.54mm:PinHeader_2x02_P2.54mm_Vertical, symbol Connector_Generic:Conn_02x02_Odd_Even
- added J22: Conn_01x03_Male_Power, Connector_PinHeader_2.54mm:PinHeader_1x03_P2.54mm_Vertical, symbol Connector:Conn_01x03_Male
- added J25: Conn_Galvo_A, Connector_PinHeader_2.54mm:PinHeader_1x03_P2.54mm_Vertical, symbol Connector:Conn_01x03_Male
- added J26: Conn_Galvo_B, Connector_PinHeader_2.54mm:PinHeader_1x03_P2.54mm_Vertical, symbol Connector:Conn_01x03_Male
- added J27: Conn_01x40_Male, Connector_PinHeader_2.54mm:PinHeader_2x20_P2.54mm_Vertical, symbol Connector:Conn_01x40_Male
- added R46: (no value), symbol Device:R_Small_US
- added R47: R_Small_US, symbol Device:R_Small_US
- added TP1, TP2, TP3, TP4, TP5: (no value), symbol Connector:TestPoint
- added U15: TLV3201, Package_TO_SOT_SMD:SOT-23-5, symbol project:TLV3201
Connections:
- net +15V: now also J22.3 (Pin_3)
- net +3V3: now also C11.1, C12.1, J27.1 (Pin_1), J27.17 (Pin_17)
- net +5V: now also C10.1, C13.1, J27.2 (Pin_2), J27.4 (Pin_4), R46.1, U15.5 (V+)
- net -15V: now also J22.1 (Pin_1)
- net GND: now also C10.2, C11.2, C12.2, C13.2, J14.2 (Pin_2), J15.2 (Pin_2), J19.1 (Pin_1), J19.3 (Pin_3), J20.2 (Pin_2), J22.2 (Pin_2), J25.1 (Pin_1), J26.1 (Pin_1), J27.14 (Pin_14), J27.20 (Pin_20), J27.25 (Pin_25), J27.30 (Pin_30), J27.34 (Pin_34), J27.39 (Pin_39), J27.6 (Pin_6), J27.9 (Pin_9), R47.2, U15.2 (V-)
- net LED_trigger: now also TP2.1
- net at U2.3 (+): now also J16.2 (Pin_2); no longer J2.1 (Pin_1)
- net at R18.1: now also J21.4 (Pin_4); no longer J6.3 (Pin_3)
- net at J2.3 (Pin_3): now also J14.3 (Pin_3), J16.3 (Pin_3); no longer U2.5 (+)
- net at C7.1, R42.1, U14.1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: now also TP4.1
- net at R36.2, U4.7: now also J23.1 (Pin_1); no longer J10.3 (Pin_3)
- net at J4.4 (Pin_4), U8.4: now also TP1.1
- net at R35.2, U5.7: now also J24.3 (Pin_3); no longer J9.2 (Pin_2)
- net at R34.2, U1.7: now also J24.1 (Pin_1); no longer J9.3 (Pin_3)
- net at J3.24 (Pin_24), U10.12 (10_CS_MQSR), U11.12 (10_CS_MQSR): now also J27.24 (Pin_24)
- net at J3.21 (Pin_21), U10.13 (11_MOSI_CTX1), U11.13 (11_MOSI_CTX1): now also J27.21 (Pin_21)
- net at J3.19 (Pin_19), U10.14 (12_MISO_MQSL), U11.14 (12_MISO_MQSL): now also J27.19 (Pin_19)
- net at J3.23 (Pin_23), U10.20 (13_SCK_CRX1_LED), U11.20 (13_SCK_CRX1_LED): now also J27.23 (Pin_23)
- net at J3.15 (Pin_15), U10.5 (3_LRCLK2), U11.5 (3_LRCLK2)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: now also J27.15 (Pin_15)
- net at J3.7 (Pin_7), U10.6 (4_BCLK2), U11.6 (4_BCLK2)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: now also J27.7 (Pin_7)
- net at J3.32 (Pin_32), U10.7 (5_IN2), U11.7 (5_IN2): now also J27.32 (Pin_32)
- net at J3.33 (Pin_33), U10.8 (6_OUT1D), U11.8 (6_OUT1D): now also J27.33 (Pin_33)
- net at U3.5 (+): now also J17.4 (Pin_4); no longer J1.3 (Pin_3)
- net at J7.2 (Pin_2), U12.4: now also TP3.1
- net at RV5.2, RV5.3, U7.1: now also J18.1 (Pin_1); no longer J5.4 (Pin_4)
- net at A1.7 (D4): now also U15.3 (+); no longer J13.1 (Pin_1)
- net at J11.3 (Pin_3), J3.5 (Pin_5): now also J27.5 (Pin_5)
- net at J11.4 (Pin_4), J3.3 (Pin_3): now also J27.3 (Pin_3)
- net at J6.1 (Pin_1): now also J20.1 (Pin_1), J21.1 (Pin_1); no longer R16.1
- net at J3.10 (Pin_10): now also J27.10 (Pin_10)
- net at J3.11 (Pin_11): now also J27.11 (Pin_11)
- net at J3.12 (Pin_12): now also J27.12 (Pin_12)
- net at J3.13 (Pin_13): now also J27.13 (Pin_13)
- net at J3.16 (Pin_16): now also J27.16 (Pin_16)
- net at J3.18 (Pin_18): now also J27.18 (Pin_18)
- net at J3.22 (Pin_22): now also J27.22 (Pin_22)
- net at J3.26 (Pin_26): now also J27.26 (Pin_26)
- net at J3.27 (Pin_27): now also J27.27 (Pin_27)
- net at J3.28 (Pin_28): now also J27.28 (Pin_28)
- net at J3.29 (Pin_29), U13.3 (+): now also J27.29 (Pin_29)
- net at J3.31 (Pin_31): now also J27.31 (Pin_31)
- net at J3.35 (Pin_35): now also J27.35 (Pin_35)
- net at J3.36 (Pin_36): now also J27.36 (Pin_36)
- net at J3.37 (Pin_37): now also J27.37 (Pin_37)
- net at J3.38 (Pin_38): now also J27.38 (Pin_38)
- net at J3.40 (Pin_40): now also J27.40 (Pin_40)
- net at J3.8 (Pin_8): now also J27.8 (Pin_8)
- net at R37.2, U5.1: now also J23.3 (Pin_3); no longer J10.2 (Pin_2)
- net at RV6.2, RV6.3, U7.7: now also J18.3 (Pin_3); no longer J5.2 (Pin_2)
- net at J12.2 (Pin_2), R42.2, R43.1: now also TP5.1
- net at J1.1 (Pin_1): now also J15.1 (Pin_1), J17.1 (Pin_1); no longer U3.3 (+)
- new net: J14.1 (Pin_1), J16.1 (Pin_1), J2.1 (Pin_1)
- new net: J24.2 (Pin_2), J25.3 (Pin_3), J9.3 (Pin_3)
- new net: J24.4 (Pin_4), J25.2 (Pin_2), J9.2 (Pin_2)
- new net: J18.4 (Pin_4), J19.2 (Pin_2), J5.2 (Pin_2)
- new net: J18.2 (Pin_2), J19.4 (Pin_4), J5.4 (Pin_4)
- new net: J16.4 (Pin_4), U2.5 (+)
- new net: J21.2 (Pin_2), R16.1
- new net: J20.3 (Pin_3), J21.3 (Pin_3), J6.3 (Pin_3)
- new net: R46.2, R47.1, U15.1 (-)
- new net: J17.2 (Pin_2), U3.3 (+)
- new net: J1.3 (Pin_3), J15.3 (Pin_3), J17.3 (Pin_3)
- new net: J10.3 (Pin_3), J23.2 (Pin_2), J26.3 (Pin_3)
- new net: J10.2 (Pin_2), J23.4 (Pin_4), J26.2 (Pin_2)
- new net: J13.1 (Pin_1), U15.4
Other:
- moved on the sheet: A1, C1, C2, C3, C4, C5, C6, C7, C8, C9, FB1, FB2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

Commit message: First PCB placement
Parts:
- C10, C12, C13: value C_Small -> (none)
- J14: value Conn_POS_input_A -> (none); footprint Connector_PinHeader_2.54mm:PinHeader_1x03_P2.54mm_Vertical -> (none)
- J15: value Conn_POS_input_B -> (none); footprint Connector_PinHeader_2.54mm:PinHeader_1x03_P2.54mm_Vertical -> (none)
- J19: value Conn_ADC -> (none)
- J20: value Conn_ADC -> (none); footprint Connector_PinHeader_2.54mm:PinHeader_1x03_P2.54mm_Vertical -> (none)
- J21, J23, J24: value Conn_02x02_Odd_Even -> (none); footprint Connector_PinHeader_2.54mm:PinHeader_2x02_P2.54mm_Vertical -> (none)
- J22: value Conn_01x03_Male_Power -> (none); footprint Connector_PinHeader_2.54mm:PinHeader_1x03_P2.54mm_Vertical -> (none)
- J25: value Conn_Galvo_A -> (none); footprint Connector_PinHeader_2.54mm:PinHeader_1x03_P2.54mm_Vertical -> (none)
- J26: value Conn_Galvo_B -> (none); footprint Connector_PinHeader_2.54mm:PinHeader_1x03_P2.54mm_Vertical -> (none)
- J27: value Conn_01x40_Male -> (none); footprint Connector_PinHeader_2.54mm:PinHeader_2x20_P2.54mm_Vertical -> (none)
- Q2: value 2N2219 -> (none); footprint Package_TO_SOT_THT:TO-39-3 -> (none)
- R45, R47: value R_Small_US -> (none)
- U15: value TLV3201 -> (none); footprint Package_TO_SOT_SMD:SOT-23-5 -> (none)
Connections:
- net at C6.1, R41.2, U14.3 (+): no longer C7.2
- net at R40.2, R41.1: now also C7.2
