File: brass_board/PCB/main_board/main_board.kicad_sch (KiCad schematic)
At the start: 146 parts

Commit message: Fix pin mis-route. Refactor schematic.
Teensy was connected to wrong audio board pins for I2S TX and RX. Fixed.

Refactored schematic using busses.

Added logical schematic symbol for Jetson header.
Parts:
- removed J27, J3: (no value), symbol Connector:Conn_01x40_Male
- added J27, J3: Jetson_HDR_40, Connector_PinHeader_2.54mm:PinHeader_2x20_P2.54mm_Vertical, symbol Jetson:Jetson_HDR_40
- C1, C12, C13, C2, C3, C4, C8, C9: value (none) -> .01u; footprint (none) -> Capacitor_SMD:C_0603_1608Metric
- C10, C11: value (none) -> 1u; footprint (none) -> Capacitor_SMD:C_0603_1608Metric
- C14, C15, C16, C17, C18, C19, C20, C21: value (none) -> 100uF; footprint (none) -> Capacitor_SMD:C_1210_3225Metric
- C5: value (none) -> .0047u; footprint (none) -> Capacitor_SMD:C_0603_1608Metric
- C6: value (none) -> 330p; footprint (none) -> Capacitor_SMD:C_0603_1608Metric
- C7: value (none) -> .0022u; footprint (none) -> Capacitor_SMD:C_0603_1608Metric
- Cam_Input1, Cam_Output1, GalvoA_Gain1, GalvoA_Offset1, GalvoB_Gain1, GalvoB_Offset1, InputA_Gain1, InputA_offset1, InputB_Gain1, InputB_offset1, LED_Trigger1, Prog1: value (none) -> 50k; footprint (none) -> Potentiometer_THT:Potentiometer_Bourns_3296W_Vertical
- D1: value (none) -> PEWPEWPEW; footprint (none) -> Diode_SMD:D_0603_1608Metric
- D2: value (none) -> Clear Fault; footprint (none) -> Diode_SMD:D_0603_1608Metric
- D3: value (none) -> LAZOR?; footprint (none) -> Diode_SMD:D_0603_1608Metric
- D4: value (none) -> LAZOR!!!; footprint (none) -> Diode_SMD:D_0603_1608Metric
- D5: value (none) -> Fault; footprint (none) -> Diode_SMD:D_0603_1608Metric
- FB1, FB2, FB3: value (none) -> GZ2012D601TF; footprint (none) -> Resistor_SMD:R_0805_2012Metric
- J1, J15: value (none) -> Conn_POS_input_B; footprint (none) -> Connector_PinHeader_2.54mm:PinHeader_1x03_P2.54mm_Vertical
- J10, J26: value (none) -> Conn_Galvo_B; footprint (none) -> Connector_PinHeader_2.54mm:PinHeader_1x03_P2.54mm_Vertical
- J11: value (none) -> Conn_OLED; footprint (none) -> Connector_PinHeader_2.54mm:PinHeader_1x04_P2.54mm_Vertical
- J12: value (none) -> Conn_LED_CTL; footprint (none) -> Connector_PinHeader_2.54mm:PinHeader_1x02_P2.54mm_Vertical
- J13: value (none) -> Conn_Laser_Trigger; footprint (none) -> Connector_PinHeader_2.54mm:PinHeader_1x02_P2.54mm_Vertical
- J14, J2: value (none) -> Conn_POS_input_A; footprint (none) -> Connector_PinHeader_2.54mm:PinHeader_1x03_P2.54mm_Vertical
- J16, J17, J18, J21, J23, J24: value (none) -> Conn_02x02_Odd_Even; footprint (none) -> Connector_PinHeader_2.54mm:PinHeader_2x02_P2.54mm_Vertical
- J19: value (none) -> Conn_ADC; footprint (none) -> Connector_PinHeader_2.54mm:PinHeader_1x04_P2.54mm_Vertical
- J20, J6: value (none) -> Conn_DAC; footprint (none) -> Connector_PinHeader_2.54mm:PinHeader_1x03_P2.54mm_Vertical
- J22: value (none) -> Conn_01x03_Amp_power; footprint (none) -> Connector_PinHeader_2.54mm:PinHeader_1x03_P2.54mm_Vertical
- J25, J9: value (none) -> Conn_Galvo_A; footprint (none) -> Connector_PinHeader_2.54mm:PinHeader_1x03_P2.54mm_Vertical
- J28: value (none) -> Conn_01x06_FTDI; footprint (none) -> Connector_PinHeader_2.54mm:PinHeader_1x06_P2.54mm_Vertical
- J4: value (none) -> Conn_01x04_Cam_Trigger; footprint (none) -> Connector_PinHeader_2.54mm:PinHeader_1x04_P2.54mm_Vertical
- J5: value (none) -> Conn_ADC; footprint (none) -> Connector_PinHeader_2.54mm:PinHeader_2x02_P2.54mm_Vertical
- J7: value (none) -> Conn_LED_PWM; footprint (none) -> Connector_PinHeader_2.54mm:PinHeader_1x02_P2.54mm_Vertical
- J8: value (none) -> Conn_Galvo_Power; footprint (none) -> Connector_PinHeader_2.54mm:PinHeader_1x03_P2.54mm_Vertical
- Q1: value (none) -> MMBT3904; footprint (none) -> Package_TO_SOT_SMD:SOT-23
- R1, R13, R14, R2, R20, R21, R22, R23, R24, R25, R26, R27, R28, R29, R3, R30, R31, R32, R33, R34, R35, R36, R37, R4, R48, R49, R5, R50, R51, R6, R7, R8: value (none) -> 1k; footprint (none) -> Resistor_SMD:R_0603_1608Metric
- R10, R11, R12, R16, R17, R18, R19, R39, R9: value (none) -> 12k; footprint (none) -> Resistor_SMD:R_0603_1608Metric
- R15, R38: value (none) -> 4.7k; footprint (none) -> Resistor_SMD:R_0603_1608Metric
- R40: value (none) -> 110k; footprint (none) -> Resistor_SMD:R_0603_1608Metric
- R41: value (none) -> 36k; footprint (none) -> Resistor_SMD:R_0603_1608Metric
- R42: value (none) -> 1.4k; footprint (none) -> Resistor_SMD:R_0603_1608Metric
- R43: value (none) -> 2.8k; footprint (none) -> Resistor_SMD:R_0603_1608Metric
- R44, R45, R46, R47, R56: value (none) -> 220; footprint (none) -> Resistor_SMD:R_0603_1608Metric
- S1: value (none) -> Reset; footprint (none) -> Project:SW_PTS525SM15SMTR2LFS
- TP1: value (none) -> Cam_Out; footprint (none) -> Connector_PinHeader_2.54mm:PinHeader_1x01_P2.54mm_Vertical
- TP2: value (none) -> LED_trigger; footprint (none) -> Connector_PinHeader_2.54mm:PinHeader_1x01_P2.54mm_Vertical
- TP3: value (none) -> TestPoint; footprint (none) -> Connector_PinHeader_2.54mm:PinHeader_1x01_P2.54mm_Vertical
- TP4: value (none) -> PWM_DAC_Out; footprint (none) -> Connector_PinHeader_2.54mm:PinHeader_1x01_P2.54mm_Vertical
- TP5: value (none) -> LED_CTL; footprint (none) -> Connector_PinHeader_2.54mm:PinHeader_1x01_P2.54mm_Vertical
- U1, U14, U2, U3, U4, U5, U6, U7: value (none) -> LM358DT; footprint (none) -> Package_SO:SOIC-8-1EP_3.9x4.9mm_P1.27mm_EP2.29x3mm
- U10, U11: value (none) -> Teensy4.0; footprint (none) -> teensy:Teensy40
- U12, U13, U8, U9: value (none) -> TLV3201; footprint (none) -> Package_TO_SOT_SMD:SOT-23-5
- U15: value (none) -> 74LS08; footprint (none) -> Package_SO:SOIC-14_3.9x8.7mm_P1.27mm
- U16: value (none) -> ARDUINO_PRO_MINI; footprint (none) -> Project:MODULE_ARDUINO_PRO_MINI
- U17: value (none) -> 74LVC1G34; footprint (none) -> Package_TO_SOT_SMD:SOT-23-5
- U18: value (none) -> TXS0102DCT; footprint (none) -> Package_SO:SSOP-8_2.95x2.8mm_P0.65mm
Connections:
- net +3V3: now also J11.3 (Pin_3), J27.1 (3V3), J27.17 (3V3), J3.1 (3V3), J3.17 (3V3); no longer J11.2 (Pin_2)
- net +5V: now also J27.2 (5V), J27.4 (5V), J3.2 (5V), J3.4 (5V)
- net GND: now also J11.4 (Pin_4), J27.14 (GND), J27.20 (GND), J27.25 (GND), J27.30 (GND), J27.34 (GND), J27.39 (GND), J27.6 (GND), J27.9 (GND), J3.14 (GND), J3.20 (GND), J3.25 (GND), J3.30 (GND), J3.34 (GND), J3.39 (GND), J3.6 (GND), J3.9 (GND); no longer J11.1 (Pin_1)
- net Prog_Reset: now also J27.29 (GPIO01), J3.29 (GPIO01)
- net SGT_RX: now also U11.10 (8_TX2_IN1); no longer U11.12 (10_CS_MQSR)
- net SGT_TX: now also U11.9 (7_RX2_OUT1A); no longer U11.11 (9_OUT1C)
- net CS: now reaches U10.12 (10_CS_MQSR)
- net CS: now also J27.24 (SPI0_CS0), J3.24 (SPI0_CS0)
- net MISO: now reaches U10.13 (11_MOSI_CTX1)
- net MISO: now also J27.21 (SPI0_MISO), J3.21 (SPI0_MISO)
- net MOSI: now reaches U10.14 (12_MISO_MQSL)
- net MOSI: now also J27.19 (SPI0_MOSI), J3.19 (SPI0_MOSI)
- net SCK: now reaches U10.20 (13_SCK_CRX1_LED)
- net SCK: now also J27.23 (SPI0_SCK), J3.23 (SPI0_SCK)
- net CAM_TRIGGER: now reaches U10.5 (3_LRCLK2), U8.3 (+)
- net CAM_TRIGGER: now also J27.15 (GPIO12), J3.15 (GPIO12)
- net CAM_EXPOSURE: now reaches U10.6 (4_BCLK2), U9.4
- net CAM_EXPOSURE: now also J27.7 (GPIO09), J3.7 (GPIO09)
- net MISC1: now reaches U10.7 (5_IN2)
- net MISC1: now also J27.32 (GPIO07), J3.32 (GPIO07)
- net MISC0: now reaches U10.8 (6_OUT1D)
- net MISC0: now also J27.33 (GPIO13), J3.33 (GPIO13)
- net LAZOR? renamed Laz0r?
- net Veapons Hot renamed Veapons_Hot
- net Veapons_Hot: now also J27.31 (GPIO11), J3.31 (GPIO11)
- new net: J27.10 (UART1_RX), J3.10 (UART1_RX)
- new net: J27.11 (UART1_RTS), J3.11 (UART1_RTS)
- new net: J27.12 (I2S0_SCLK), J3.12 (I2S0_SCLK)
- new net: J27.13 (SPI1_SCK), J3.13 (SPI1_SCK)
- new net: J27.16 (SPI1_CS1), J3.16 (SPI1_CS1)
- new net: J27.18 (SPI1_CS0), J3.18 (SPI1_CS0)
- new net: J27.22 (SPI1_MISO), J3.22 (SPI1_MISO)
- new net: J27.26 (SPI0_CS1), J3.26 (SPI0_CS1)
- new net: J27.27 (I2C0_SDA), J3.27 (I2C0_SDA)
- new net: J27.28 (I2C0_SCL), J3.28 (I2C0_SCL)
- new net: J27.35 (I2S0_FS), J3.35 (I2S0_FS)
- new net: J27.36 (UART1_CTS), J3.36 (UART1_CTS)
- new net: J27.37 (SPI1_MOSI), J3.37 (SPI1_MOSI)
- new net: J27.38 (I2S0_SDIN), J3.38 (I2S0_SDIN)
- new net: J27.40 (I2S_SDOUT), J3.40 (I2S_SDOUT)
- new net: J27.8 (UART1_TX), J3.8 (UART1_TX)
- new net OLED_SCL: J11.2 (Pin_2), J27.5 (I2C1_SCL), J3.5 (I2C1_SCL)
- new net OLED_SDA: J11.1 (Pin_1), J27.3 (I2C1_SDA), J3.3 (I2C1_SDA)
- no-connect marks 0 -> 23
Other:
- note added: "MISO/MOSI are swapped here ON PURPOSE ->"
- moved on the sheet: D2, D3, D4, D5, J11, Prog1, Q1, R38, R45, R46, R47, R56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

Commit message: Big PCB update: Added LED driver, Added laser interface, Fixed errors from RC1
Parts:
- added C22, C23, C24, C25, C26, C28, C29, C? (x9): 100uF, Capacitor_SMD:C_1210_3225Metric, symbol Device:C_Small
- added C27, C?, R61, R?: 4.7uF, Capacitor_SMD:C_0603_1608Metric, symbol Device:C_Small
- added C30, C?: 22uF, Capacitor_SMD:C_2220_5650Metric, symbol Device:C_Small
- added C? (x2): 330p, Capacitor_SMD:C_0603_1608Metric, symbol Device:C_Small
- added C?: .0022u, Capacitor_SMD:C_0603_1608Metric, symbol Device:C_Small
- added C? (x4): 0.1u, Capacitor_SMD:C_0603_1608Metric, symbol Device:C_Small
- added C?: .0047u, Capacitor_SMD:C_0603_1608Metric, symbol Device:C_Small
- added C? (x2): .01u, Capacitor_SMD:C_0603_1608Metric, symbol Device:C_Small
- added D6, D?: PD3100, Diode_SMD:D_PowerDI-5, symbol Diode:CDBA3100-HF
- added D?: BZV55B3V3, Diode_SMD:D_MiniMELF, symbol Diode:BZV55B3V3
- added D?: Ready, Diode_SMD:D_0603_1608Metric, symbol Device:LED
- added D?: Danger, Diode_SMD:D_0603_1608Metric, symbol Device:LED
- added D?: Veapons_Hot, Diode_SMD:D_0603_1608Metric, symbol Device:LED
- added H1, H2, H3, H4: MountingHole, MountingHole:MountingHole_3.2mm_M3, symbol Mechanical:MountingHole
- added J29, J?: Conn_LED_Power, Connector_Molex:Molex_KK-254_AE-6410-02A_1x02_P2.54mm_Vertical, symbol Connector:Conn_01x02_Male
- added J30: DB25_Female_MountingHoles, Connector_Dsub:DSUB-25_Female_Horizontal_P2.77x2.84mm_EdgePinOffset4.94mm_Housed_MountingHolesOffset7.48mm, symbol Connector:DB25_Female_MountingHoles
- added J?: Danger, Connector_Molex:Molex_KK-254_AE-6410-02A_1x02_P2.54mm_Vertical, symbol Connector:Conn_01x02_Male
- added J?: RS232, Connector_PinHeader_2.54mm:PinHeader_2x02_P2.54mm_Vertical, symbol Connector_Generic:Conn_02x02_Odd_Even
- added J?: Stop, Connector_Molex:Molex_KK-254_AE-6410-02A_1x02_P2.54mm_Vertical, symbol Connector:Conn_01x02_Male
- added J?: Ready, Connector_Molex:Molex_KK-254_AE-6410-02A_1x02_P2.54mm_Vertical, symbol Connector:Conn_01x02_Male
- added J?: Conn_LED_Temp, Connector_PinHeader_2.54mm:PinHeader_1x02_P2.54mm_Vertical, symbol Connector:Conn_01x02_Male
- added J?: Reset, Connector_Molex:Molex_KK-254_AE-6410-02A_1x02_P2.54mm_Vertical, symbol Connector:Conn_01x02_Male
- added K?: DIPxx-1Axx-11x, Relay_THT:Relay_StandexMeder_DIP_LowProfile, symbol Relay:DIPxx-1Axx-11x
- added L1, L?: 22u, Project:CDRH74, symbol Device:L_Ferrite
- added LED_Temp?: 50k, Potentiometer_THT:Potentiometer_Bourns_3296W_Vertical, symbol Device:R_Potentiometer_US
- added Q2, Q?: AO3400A, Package_TO_SOT_SMD:SOT-23, symbol Transistor_FET:AO3400A
- added R52, R53, R54, R55, R? (x4): R_Small_US, Capacitor_SMD:C_0603_1608Metric, symbol Device:R_Small_US
- added R57, R?: 10k, Capacitor_SMD:C_0603_1608Metric, symbol Device:R_Small_US
- added R58, R?: 100k, Capacitor_SMD:C_0603_1608Metric, symbol Device:R_Small_US
- added R59, R?: 33k1, Capacitor_SMD:C_0603_1608Metric, symbol Device:R_Small_US
- added R60, R?: 4.7nF1, Capacitor_SMD:C_0603_1608Metric, symbol Device:C_Small
- added R62, R?: 0.147, Resistor_SMD:R_1206_3216Metric, symbol Device:R_Small_US
- added R?: 36k, Resistor_SMD:R_0603_1608Metric, symbol Device:R_Small_US
- added R? (x4): 1k, Resistor_SMD:R_0603_1608Metric, symbol Device:R_Small_US
- added R? (x2): 330k, Capacitor_SMD:C_0603_1608Metric, symbol Device:R_Small_US
- added R?: 12k, Resistor_SMD:R_0603_1608Metric, symbol Device:R_Small_US
- added R? (x3): --, Capacitor_SMD:C_0603_1608Metric, symbol Device:R_Small_US
- added R?: 3.3M, Resistor_SMD:R_0603_1608Metric, symbol Device:R_Small_US
- added R?: 470k, Resistor_SMD:R_0603_1608Metric, symbol Device:R_Small_US
- added R? (x2): 390k, Capacitor_SMD:C_0603_1608Metric, symbol Device:R_Small_US
- added R?: 91k, Resistor_SMD:R_0603_1608Metric, symbol Device:R_Small_US
- added R?: 47k, Resistor_SMD:R_0603_1608Metric, symbol Device:R_Small_US
- added R?: 110k, Resistor_SMD:R_0603_1608Metric, symbol Device:R_Small_US
- added R?: 440, Resistor_SMD:R_0603_1608Metric, symbol Device:R_Small_US
- added S?: Reset, Project:SW_PTS525SM15SMTR2LFS, symbol project:PTS525SM15SMTR2LFS
- added TP?: TestPoint, Connector_PinHeader_2.54mm:PinHeader_1x01_P2.54mm_Vertical, symbol Connector:TestPoint
- added TP?: LED_Temp, Connector_PinHeader_2.54mm:PinHeader_1x01_P2.54mm_Vertical, symbol Connector:TestPoint
- added U19, U?: LT3956, Project:CONV_LT3958EUHE#PBF, symbol project:LT3956
- added U?: SP3232E, Package_SO:HTSSOP-16-1EP_4.4x5mm_P0.65mm_EP3x3mm, symbol project:SP3232E
- added U? (x3): LM358, symbol Amplifier_Operational:LM358
- added U? (x5): TXS0102DCT, Package_SO:SSOP-8_2.95x2.8mm_P0.65mm, symbol Logic_LevelTranslator:TXS0102DCT
- added U? (x2): TCA9535PWR, Project:SOP65P640X120-24N, symbol project:TCA9535PWR
- added U?: TLV3201, Package_TO_SOT_SMD:SOT-23-5, symbol project:TLV3201
- J10, J9: footprint Connector_PinHeader_2.54mm:PinHeader_1x03_P2.54mm_Vertical -> Connector_JST:JST_XH_B3B-XH-A_1x03_P2.50mm_Vertical
- J8: footprint Connector_PinHeader_2.54mm:PinHeader_1x03_P2.54mm_Vertical -> Connector_Molex:Molex_KK-254_AE-6410-03A_1x03_P2.54mm_Vertical
- R1, R2, R22, R23, R24, R25, R26, R27, R28, R29, R3, R30, R31, R32, R33, R34, R35, R36, R37, R4, R5, R6, R7, R8: value 1k -> 10k; LCSC C21190 -> (none)
- R15: value 4.7k -> 560
- R44, R45, R46, R47, R56: value 220 -> 440; LCSC C22962 -> (none)
- R48, R49, R50, R51: value 1k -> 5k; LCSC C21190 -> (none)
Connections:
- net +15V: now also R15.1, C?.1, C?.1, U?.8 (V+)
- net +3V3: now also J?.1 (Pin_1), LED_Temp?.1, U?.16 (VCC), U?.21 (A0), U?.24 (VCC), U?.24 (VCC), U?.3 (VCCA), U?.3 (VCCA), U?.3 (VCCA), U?.3 (VCCA), U?.3 (VCCA), U?.5 (V+), U?.6 (OE), U?.6 (OE), U?.6 (OE), U?.6 (OE), U?.6 (OE); no longer R15.1
- net +5V: now also U?.7 (VCCB), U?.7 (VCCB), U?.7 (VCCB), U?.7 (VCCB), U?.7 (VCCB)
- net -15V: now also C?.2, C?.2, U?.4 (V-)
- net Cam_In: now also U8.1; no longer U8.4
- net GND: now also C?.1, C?.1, C?.1, C?.2, C?.2, C?.2, C?.2, C?.2, C?.2, D?.1 (K), D?.1 (K), D?.2 (A), J30.0 (PAD), J30.1, J30.2, J30.24 (P24), J30.9, J?.1 (Pin_1), J?.1 (Pin_1), J?.1 (Pin_1), K?.1, K?.14, LED_Temp?.3, R?.1, R?.2, S?.1, S?.2, U?.12 (GND), U?.12 (GND), U?.15 (GND), U?.2 (A1), U?.2 (A1), U?.2 (GND), U?.2 (GND), U?.2 (GND), U?.2 (GND), U?.2 (GND), U?.2 (V-), U?.21 (A0), U?.3 (A2), U?.3 (A2); no longer U15.10, U15.12, U15.13, U15.9
- net LED_trigger: now also J27.7 (GPIO09), J3.7 (GPIO09), U10.6 (4_BCLK2), U12.4 (-), U9.1, R?.1; no longer J4.3 (Pin_3), R15.2, U12.1 (-), U9.3 (+)
- net Veapons_Hot: now also R?.2
- net at Cam_Output1.2: now also R?.2; no longer U9.1 (-)
- net Laser_Trigger: now reaches U10.11 (9_OUT1C)
- net Laser_PWM_DAC: now reaches U10.21 (14_A0_TX3_SPDIF_OUT)
- net Laser_PWM_DAC: now also R?.1
- net Red_Laser_Trigger: now reaches U10.29 (22_A8_CTX1)
- net Jetson_RX: now reaches J27.10 (UART1_RX), J3.10 (UART1_RX)
- net Jetson_RX: now also U?.12 (R1OUT)
- net I/O_SDA: now reaches J27.27 (I2C0_SDA), J3.27 (I2C0_SDA)
- net I/O_SDA: now also U?.23 (SDA), U?.23 (SDA)
- net I/O_SCL: now reaches J27.28 (I2C0_SCL), J3.28 (I2C0_SCL)
- net I/O_SCL: now also U?.22 (SCL), U?.22 (SCL)
- net Jetson_TX: now reaches J27.8 (UART1_TX), J3.8 (UART1_TX)
- net Jetson_TX: now also U?.11 (T1IN)
- net LED_PWM: now reaches J7.2 (Pin_2), TP3.1
- net LED_PWM: now also U12.1, U15.12, U15.9; no longer U12.4
- net at U15.11: now also U?.33 (PWM)
- net at R38.1: now also U13.1; no longer U13.4
- net at Cam_Input1.2: now also U8.4 (-); no longer U8.1 (-)
- net at Prog1.2: now also U13.4 (-); no longer U13.1 (-)
- net LED_CTL: now reaches J12.2 (Pin_2), R42.2, R43.1, TP5.1
- net LED_CTL: now also U19.31 (CTRL), U?.31 (CTRL)
- net at U15.8: now also U19.33 (PWM)
- removed net CAM_EXPOSURE: J27.7 (GPIO09), J3.7 (GPIO09), U10.6 (4_BCLK2), U9.4
- net PWM_DAC renamed LED_PWM_DAC
- new net: C22.1, C23.1, C24.1, C25.1, C26.1, C28.1, C29.1, L1.1, R52.1, U19.6 (Vin)
- new net: D6.2 (A), L1.2, U19.20 (SW), U19.21 (SW), U19.8 (SW), U19.9 (SW)
- new net: C?.2, R?.1, R?.2 (x2)
- new net: C?.1, R?.2, U?.3 (+)
- new net: C?.1, C?.1, C?.1, C?.1, C?.1, C?.1, C?.1, L?.1, R?.1, U?.6 (Vin)
- new net: J?.2 (Pin_2), R?.1 (x2)
- new net: C?.1, U?.1 (C1+)
- new net: J?.3 (Pin_3), U?.13 (R1IN)
- new net: J?.1 (Pin_1), U?.14 (T1OUT)
- new net: C?.1, U?.2 (V+)
- new net: C?.2, U?.3 (C1-)
- new net: C?.1, U?.4 (C2+)
- new net: C?.2, U?.5 (C2-)
- new net: C?.1, U?.6 (V-)
- new net: C27.1, U19.35 (SS)
- new net: R?.1, R?.2, U?.3 (intVcc)
- new net: U?.4 (A2), U?.7 (P03)
- new net: U?.5 (A1), U?.6 (P02)
- new net: Q?.1 (G), U?.23 (PWMout)
- new net: J?.1 (Pin_1), Q?.3 (D)
- new net: U?.4 (A2), U?.9 (P05)
- new net: U?.5 (A1), U?.8 (P04)
- new net: R?.1, R?.2, U?.2 (EN/UVLO)
- new net: D?.2 (A), R?.1 (x3)
- new net: J?.1 (Pin_1), K?.2, R?.2, R?.2
- new net: R?.1, R?.2, U9.4 (-)
- new net: C?.1, U?.35 (SS)
- new net: R59.2, R60.1
- new net: C?.2, R?.1, R?.1, U?.12 (PGND), U?.13 (PGND), U?.14 (PGND), U?.15 (PGND), U?.16 (PGND), U?.17 (PGND), U?.28 (ISP)
- new net: J?.2 (Pin_2), R?.2, U?.27 (ISN)
- new net: R?.1, R?.2, U?.25 (FB)
- new net: C?.1, U?.1, U?.2 (-), U?.5 (+)
- new net: R?.1, U?.36 (RT)
- new net: R58.2, R61.1, U19.3 (intVcc)
- new net: D?.1 (K), J30.23 (P23), J?.2 (Pin_2), K?.6, K?.7, K?.8, S?.3, S?.4
- new net: C30.1, D6.1 (K)
- new net: C30.2, R54.1, R62.1, U19.12 (PGND), U19.13 (PGND), U19.14 (PGND), U19.15 (PGND), U19.16 (PGND), U19.17 (PGND), U19.28 (ISP)
- new net: R52.2, R53.1, U19.2 (EN/UVLO)
- new net: J29.1 (Pin_1), Q2.3 (D)
- new net: J29.2 (Pin_2), R62.2, U19.27 (ISN)
- new net: J?.2 (Pin_2), R?.1, TP?.1, U?.3 (+)
- new net: U?.4 (A2), U?.5 (P01)
- new net: U?.4 (P00), U?.5 (A1)
- new net: R58.1, R?.1, U19.34 (~VMODE)
- new net: R?.1, R?.2
- new net: R54.2, R55.1, U19.25 (FB)
- new net: LED_Temp?.2, R?.1
- new net: R?.1, R?.2, U?.4 (-)
- new net: R?.1, R?.2, U?.6 (-)
- new net: Q2.1 (G), U19.23 (PWMout)
- new net: D?.2 (A), L?.2, U?.20 (SW), U?.21 (SW), U?.8 (SW), U?.9 (SW)
- new net: R57.1, U19.36 (RT)
- new net: R59.1, U19.30 (Vc)
- new net: R?.1, R?.1, U?.34 (~VMODE)
- new net: C?.1, D?.1 (K)
- new net: R?.1, U?.30 (Vc)
- new net Cam_Out: C?.1, D?.1 (K), J4.3 (Pin_3), R15.2, U9.3 (+)
- new net Current_Alarm_TTL: J30.19 (P19), U?.1 (B2)
- new net GND2: C22.2, C23.2, C24.2, C25.2, C26.2, C27.2, C28.2, C29.2, C?.2, C?.2, C?.2, C?.2, C?.2, C?.2, C?.2, C?.2, Q2.2 (S), Q?.2 (S), R53.2, R55.2, R57.2, R60.2, R61.2, R?.2, R?.2, R?.2, R?.2, R?.2, R?.2, R?.2, U19.24 (GND), U19.4 (GND), U?.24 (GND), U?.4 (GND)
- new net LED_A_On: U15.13, U?.14 (P11)
- new net LED_B_On: U15.10, U?.13 (P10)
- new net LED_Open_Fault_A: R?.1, R?.2, U?.16 (P13)
- new net LED_Open_Fault_B: R?.1, R?.2, U?.15 (P12)
- new net LED_Temp_Fault: R?.2, TP?.1, U?.1, U?.17 (P14)
- new net Laser_Interlock: J?.2 (Pin_2), R?.2, R?.2, U?.8 (B1)
- new net Laser_PWM_DAC_0-5v: J30.8, R?.2, U?.7
- new net Laser_RX: J30.5, J?.2 (Pin_2)
- new net Laser_TX: J30.4, J?.4 (Pin_4)
- new net Laser_Trigger_TTL: J30.17 (P17)
- new net Red_Laser_Trigger_TTL: J30.15 (P15)
- new net Simmer_Control_TTL: J30.22 (P22), U?.1 (B2)
- new net System_Alarm_TTL: J30.14 (P14), U?.8 (B1)
- new net Temp_Alarm_TTL: J30.20 (P20), U?.8 (B1)
- no-connect marks 23 -> 21
Other:
- note added: "G = 1 + R2/R1 5/3.3 = 1.5151 R2/R1 = 0.5151 91k/47k = 0.5164"
- note added: "Hardware"
- note added: "LED Driver"
- note added: "Laser Interface"
- note added: "R1"
- note added: "R2"
- note added: "Ron = 160ohm max 25ma max 15V/25ma = 600 ohm 600 - 160 = 440 ohm | 20% safety: 530 ohm E12 value: 560 ohm 15V/720ohm = 21ma"
- moved on the sheet: C1, C10, C11, C12, C13, C14, C15, C16, C17, C18, C19, C2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

Commit message: main board updates
Parts:
- removed C28, C29, C? (x7): 100uF, Capacitor_SMD:C_1210_3225Metric, symbol Device:C_Small
- removed C30, C?: 22uF, Capacitor_SMD:C_2220_5650Metric, symbol Device:C_Small
- removed C?, R61, R?: 4.7uF, Capacitor_SMD:C_0603_1608Metric, symbol Device:C_Small
- removed D6, D?: PD3100, Diode_SMD:D_PowerDI-5, symbol Diode:CDBA3100-HF
- removed J12: Conn_LED_CTL, Connector_PinHeader_2.54mm:PinHeader_1x02_P2.54mm_Vertical, symbol Connector:Conn_01x02_Male
- removed J13: Conn_Laser_Trigger, Connector_PinHeader_2.54mm:PinHeader_1x02_P2.54mm_Vertical, symbol Connector:Conn_01x02_Male
- removed J29, J?: Conn_LED_Power, Connector_Molex:Molex_KK-254_AE-6410-02A_1x02_P2.54mm_Vertical, symbol Connector:Conn_01x02_Male
- removed J7: Conn_LED_PWM, Connector_PinHeader_2.54mm:PinHeader_1x02_P2.54mm_Vertical, symbol Connector:Conn_01x02_Male
- removed L1, L?: 22u, Project:CDRH74, symbol Device:L_Ferrite
- removed Prog1: 50k, Potentiometer_THT:Potentiometer_Bourns_3296W_Vertical, symbol Device:R_Potentiometer_US
- removed Q2, Q?: AO3400A, Package_TO_SOT_SMD:SOT-23, symbol Transistor_FET:AO3400A
- removed R54, R55, R? (x4): R_Small_US, Capacitor_SMD:C_0603_1608Metric, symbol Device:R_Small_US
- removed R57, R?: 10k, Capacitor_SMD:C_0603_1608Metric, symbol Device:R_Small_US
- removed R58, R?: 100k, Capacitor_SMD:C_0603_1608Metric, symbol Device:R_Small_US
- removed R59, R?: 33k1, Capacitor_SMD:C_0603_1608Metric, symbol Device:R_Small_US
- removed R60, R?: 4.7nF1, Capacitor_SMD:C_0603_1608Metric, symbol Device:C_Small
- removed R62, R?: 0.147, Resistor_SMD:R_1206_3216Metric, symbol Device:R_Small_US
- removed R?: 330k, Capacitor_SMD:C_0603_1608Metric, symbol Device:R_Small_US
- removed R?: 390k, Capacitor_SMD:C_0603_1608Metric, symbol Device:R_Small_US
- removed U19, U?: LT3956, Project:CONV_LT3958EUHE#PBF, symbol project:LT3956
- removed U? (x2): TXS0102DCT, Package_SO:SSOP-8_2.95x2.8mm_P0.65mm, symbol Logic_LevelTranslator:TXS0102DCT
- removed U? (x2): TCA9535PWR, Project:SOP65P640X120-24N, symbol project:TCA9535PWR
- added DC1, DC2: LM2596S_Module, Project:LM2596S Module, symbol project:LM2596S_Module
- added J29, J38: Pow 80V max, Connector_PinHeader_2.54mm:PinHeader_1x04_P2.54mm_Vertical, symbol Connector:Conn_01x04_Male
- added J31: Conn_01x04_LED_Supply, Connector_Molex:Molex_KK-254_AE-6410-04A_1x04_P2.54mm_Vertical, symbol Connector:Conn_01x04_Male
- added J39, J40, J41, J42: Conn_01x08_Male, Connector_PinHeader_2.54mm:PinHeader_1x08_P2.54mm_Vertical, symbol Connector:Conn_01x08_Male
- added J43, J44: Pow GND, Connector_PinHeader_2.54mm:PinHeader_1x04_P2.54mm_Vertical, symbol Connector:Conn_01x04_Male
- added J45, J46: GND, Connector_PinHeader_2.54mm:PinHeader_1x04_P2.54mm_Vertical, symbol Connector:Conn_01x04_Male
- added J47, J48: Control, Connector_PinHeader_2.54mm:PinHeader_1x04_P2.54mm_Vertical, symbol Connector:Conn_01x04_Male
- added J7: Conn_02x02_Odd_Even, Connector_PinHeader_2.54mm:PinHeader_2x02_P2.54mm_Vertical, symbol Connector_Generic:Conn_02x02_Odd_Even
- added R54: 100, Resistor_SMD:R_0603_1608Metric, symbol Device:R_US
- added R92, R93: 4.7k, Resistor_SMD:R_0603_1608Metric, symbol Device:R_Small_US
- added TP8: Laser Trigger, Connector_PinHeader_2.54mm:PinHeader_1x01_P2.54mm_Vertical, symbol Connector:TestPoint
- added U23, U24: TCA9555, Project:SOP65P640X120-24N, symbol project:TCA9555
- added U31, U32, U33, U34, U35: 74LVC1G34, Package_TO_SOT_SMD:SOT-23-5, symbol project:74LVC1G34
- C22, C25: value 100uF -> 3300uF; footprint Capacitor_SMD:C_1210_3225Metric -> Capacitor_SMD:CP_Elec_18x22
- C23, C24: value 100uF -> .01u; footprint Capacitor_SMD:C_1210_3225Metric -> Capacitor_SMD:C_0603_1608Metric; LCSC (none) -> C57112; LCSL C90143 -> (none)
- C26: LCSC (none) -> C90143; LCSL C90143 -> (none)
- C27: value 4.7uF -> 100uF; footprint Capacitor_SMD:C_0603_1608Metric -> Capacitor_SMD:C_1210_3225Metric; LCSC (none) -> C90143
- J1: value Conn_POS_input_B -> (Y); footprint Connector_PinHeader_2.54mm:PinHeader_1x03_P2.54mm_Vertical -> Connector_JST:JST_XH_B3B-XH-A_1x03_P2.50mm_Vertical
- J10: value Conn_Galvo_B -> (Y)
- J2: value Conn_POS_input_A -> (X); footprint Connector_PinHeader_2.54mm:PinHeader_1x03_P2.54mm_Vertical -> Connector_JST:JST_XH_B3B-XH-A_1x03_P2.50mm_Vertical
- J32: renamed from J?; footprint Connector_PinHeader_2.54mm:PinHeader_1x02_P2.54mm_Vertical -> Connector_Molex:Molex_KK-254_AE-6410-02A_1x02_P2.54mm_Vertical; LCSC C358684 -> (none)
- J4: value Conn_01x04_Cam_Trigger -> Cam_Trigger; footprint Connector_PinHeader_2.54mm:PinHeader_1x04_P2.54mm_Vertical -> Connector_Molex:Molex_KK-254_AE-6410-04A_1x04_P2.54mm_Vertical
- J9: value Conn_Galvo_A -> (X)
- R52: value R_Small_US -> 270k
- R53: value R_Small_US -> 330k
- R74: renamed from R?; value 390k -> 270k
- S1: footprint Project:SW_PTS525SM15SMTR2LFS -> SW_PTS525SM15SMTR2LFS
- S2: renamed from S?; footprint Project:SW_PTS525SM15SMTR2LFS -> SW_PTS525SM15SMTR2LFS
- U1, U14, U2, U3, U4, U5, U6, U7: footprint Package_SO:SOIC-8-1EP_3.9x4.9mm_P1.27mm_EP2.29x3mm -> Package_SO:SOIC-8_3.9x4.9mm_P1.27mm
- U16: footprint Project:MODULE_ARDUINO_PRO_MINI -> MODULE_ARDUINO_PRO_MINI
- U29: renamed from U?; value LM358 -> LM358DT; footprint (none) -> Package_SO:SOIC-8_3.9x4.9mm_P1.27mm
- gave numbers to parts that had none: 46
Connections:
- net Laser_Trigger_TTL is gone; now on net Laser_Trigger: J30.17 (P17)
- net +15V: now also C23.1, C26.1
- net +3V3: now also U23.21 (A0), U23.24 (VCC), U24.24 (VCC)
- net +5V: now also R54.1, R92.2, U31.5 (VCC), U32.5 (VCC), U33.5 (VCC), U34.5 (VCC), U35.5 (VCC)
- net -15V: now also C24.2, C27.2
- net Cam_Out: now also J7.1 (Pin_1), J7.3 (Pin_3); no longer R15.2
- net Current_Alarm_TTL: now also U20.8 (B1), U32.4; no longer J30.19 (P19), U20.1 (B2)
- net GND: now also C22.2, C23.2, C24.1, C25.2, C26.2, C27.1, R53.2, R72.2, U17.1, U18.1 (B2), U27.10 (T2IN), U27.17 (GND), U27.8 (R2IN), DC1.2 (In(-)), DC1.3 (Out(-)), DC2.2 (In(-)), DC2.3 (Out(-)), J31.1 (Pin_1), J31.2 (Pin_2), J43.1 (Pin_1), J43.2 (Pin_2), J43.3 (Pin_3), J43.4 (Pin_4), J44.1 (Pin_1), J44.2 (Pin_2), J44.3 (Pin_3), J44.4 (Pin_4), J45.1 (Pin_1), J45.2 (Pin_2), J45.3 (Pin_3), J45.4 (Pin_4), J46.1 (Pin_1), J46.2 (Pin_2), J46.3 (Pin_3), J46.4 (Pin_4), J47.1 (Pin_1), J48.1 (Pin_1), R93.1, U23.12 (GND), U23.2 (A1), U23.3 (A2), U24.12 (GND), U24.2 (A1), U24.21 (A0), U24.3 (A2), U31.1, U31.3 (GND), U32.1, U32.3 (GND), U33.1, U33.3 (GND), U34.1, U34.3 (GND), U35.1, U35.3 (GND); no longer U11.47 (GND)
- net I/O_SCL: now also U23.22 (SCL), U24.22 (SCL)
- net I/O_SDA: now also U23.23 (SDA), U24.23 (SDA)
- net LED_A_On: now also J42.2 (Pin_2), U23.14 (P11)
- net LED_B_On: now also J42.1 (Pin_1), U23.13 (P10)
- net LED_CTL: now also J47.4 (Pin_4), J48.4 (Pin_4)
- net LED_Open_Fault_A: now also J42.4 (Pin_4), U23.16 (P13)
- net LED_Open_Fault_B: now also R52.2, R53.1, J42.3 (Pin_3), U23.15 (P12)
- net LED_Temp_Fault: now also J42.5 (Pin_5), U23.17 (P14)
- net Laser_Trigger: now also U17.4, TP8.1; no longer U10.11 (9_OUT1C)
- net Red_Laser_Trigger_TTL: now also U34.2; no longer J30.15 (P15)
- net Simmer_Control_TTL: now also U21.8 (B1), U33.2; no longer J30.22 (P22), U21.1 (B2)
- net System_Alarm_TTL: now also U20.1 (B2), U31.4; no longer J30.14 (P14), U20.8 (B1)
- net Temp_Alarm_TTL: now also U21.1 (B2), U35.4; no longer J30.20 (P20), U21.8 (B1)
- net Pos_A(+): now reaches J14.1 (Pin_1), J16.1 (Pin_1), J2.1 (Pin_1)
- net Pos_A(-): now reaches J14.3 (Pin_3), J16.3 (Pin_3), J2.3 (Pin_3)
- net at U21.4 (A2): now also J41.3 (Pin_3), U23.6 (P02)
- net at U21.5 (A1): now also J41.2 (Pin_2), U23.5 (P01)
- net at U22.5 (A1): now also J41.1 (Pin_1), U23.4 (P00)
- net at U15.11: now also J47.3 (Pin_3)
- net at U20.4 (A2): now also J41.5 (Pin_5), U23.8 (P04)
- net at U20.5 (A1): now also J41.4 (Pin_4), U23.7 (P03)
- net at U13.4 (-): now also R92.1, R93.2
- net Pos_B(+): now reaches J1.1 (Pin_1), J15.1 (Pin_1), J17.1 (Pin_1)
- net Pos_B(-): now reaches J1.3 (Pin_3), J15.3 (Pin_3), J17.3 (Pin_3)
- net at R74.1: now also J47.2 (Pin_2)
- net at U15.8: now also J48.3 (Pin_3)
- removed net GND2: C22.2, C23.2, C24.2, C25.2, C26.2, C27.2, R53.2, R72.2
- new net: DC1.4 (Out(+)), J29.1 (Pin_1), J29.2 (Pin_2), J29.3 (Pin_3), J29.4 (Pin_4)
- new net: J30.14 (P14), U31.2
- new net: J30.15 (P15), U34.4
- new net: J41.6 (Pin_6), U23.9 (P05)
- new net: J41.7 (Pin_7), U23.10 (P06)
- new net: J41.8 (Pin_8), U23.11 (P07)
- new net: J30.20 (P20), U35.2
- new net: J48.2 (Pin_2), R52.1
- new net: DC2.4 (Out(+)), J38.1 (Pin_1), J38.2 (Pin_2), J38.3 (Pin_3), J38.4 (Pin_4)
- new net: J7.4 (Pin_4), R15.2
- new net: J30.19 (P19), U32.2
- new net: J30.22 (P22), U33.4
- new net: J39.1 (Pin_1), U24.4 (P00)
- new net: J39.2 (Pin_2), U24.5 (P01)
- new net: J39.3 (Pin_3), U24.6 (P02)
- new net: J39.4 (Pin_4), U24.7 (P03)
- new net: J39.5 (Pin_5), U24.8 (P04)
- new net: J39.6 (Pin_6), U24.9 (P05)
- new net: J39.7 (Pin_7), U24.10 (P06)
- new net: J39.8 (Pin_8), U24.11 (P07)
- new net: J40.1 (Pin_1), U24.13 (P10)
- new net: J40.2 (Pin_2), U24.14 (P11)
- new net: J40.3 (Pin_3), U24.15 (P12)
- new net: J40.4 (Pin_4), U24.16 (P13)
- new net: J40.5 (Pin_5), U24.17 (P14)
- new net: J40.6 (Pin_6), U24.18 (P15)
- new net: J40.7 (Pin_7), U24.19 (P16)
- new net: J40.8 (Pin_8), U24.20 (P17)
- new net: J7.2 (Pin_2), R54.2
- new net: J42.6 (Pin_6), U23.18 (P15)
- new net: J42.7 (Pin_7), U23.19 (P16)
- new net: J42.8 (Pin_8), U23.20 (P17)
- new net +24V: C22.1, C25.1, DC1.1 (In(+)), DC2.1 (In(+)), J31.3 (Pin_3), J31.4 (Pin_4)
- no-connect marks 21 -> 95
Other:
- note added: "Ron = 160ohm max 25ma max 15V/25ma = 600 ohm 600 - 160 = 440 ohm | 20% safety: 530 ohm E12 value: 560 ohm 15V/720ohm = 21ma 5V/(160+100)ohm = 19ma"
- note removed: "Ron = 160ohm max 25ma max 15V/25ma = 600 ohm 600 - 160 = 440 ohm | 20% safety: 530 ohm E12 value: 560 ohm 15V/720ohm = 21ma"
- moved on the sheet: C1, C10, C11, C12, C13, C14, C15, C16, C17, C18, C19, C2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
