File: brass_board/PCB/main_board/main_board.kicad_sch (KiCad schematic)
At the start: 232 parts, among them J1 (Y), J10 (Y), J11 Conn_OLED, J14 Conn_POS_input_A, J15 Conn_POS_input_B, J16 Conn_02x02_Odd_Even, J17 Conn_02x02_Odd_Even, J18 Conn_02x02_Odd_Even, J19 Conn_ADC, J2 (X), J20 Conn_DAC, J21 Conn_02x02_Odd_Even, J22 Conn_01x03_Amp_power, J23 Conn_02x02_Odd_Even, J24 Conn_02x02_Odd_Even, J25 Conn_Galvo_A, J26 Conn_Galvo_B, J27 Jetson_HDR_40, J28 Conn_01x06_FTDI, J29 Pow 80V max, J3 Jetson_HDR_40, J30 DB25_Female_MountingHoles, J31 Conn_01x04_LED_Supply, J32 Conn_LED_Temp, J33 RS232, J34 Reset, J35 Danger, J36 Stop, J37 Ready, J38 Pow 80V max, J39 Conn_01x08_Male, J4 Cam_Trigger, J40 Conn_01x08_Male, J41 Conn_01x08_Male, J42 Conn_01x08_Male, J43 Pow GND, J44 Pow GND, J45 GND, J46 GND, J47 Control, J48 Control, J5 Conn_ADC, J6 Conn_DAC, J7 Conn_02x02_Odd_Even, J8 Conn_Galvo_Power, J9 (X), K1 DIPxx-1Axx-11x, Q1 MMBT3904, U1 LM358DT, U10 Teensy4.0, U11 Teensy4.0, U12 TLV3201, U13 TLV3201, U14 LM358DT, U15 74LS08, U16 ARDUINO_PRO_MINI, U17 74LVC1G34, U18 TXS0102DCT, U2 LM358DT, U20 TXS0102DCT, U21 TXS0102DCT, U22 TXS0102DCT, U23 TCA9555, U24 TCA9555, U27 SP3232E, U28 TLV3201, U29 LM358DT, U3 LM358DT, U31 74LVC1G34, U32 74LVC1G34, U33 74LVC1G34, U34 74LVC1G34, U35 74LVC1G34, U4 LM358DT, U5 LM358DT, U6 LM358DT, U7 LM358DT, U8 TLV3201, U9 TLV3201

Commit message: Updates to main board
Parts:
- removed J19: Conn_ADC, Connector_PinHeader_2.54mm:PinHeader_1x04_P2.54mm_Vertical, symbol Connector:Conn_01x04_Male
- removed J5: Conn_ADC, Connector_PinHeader_2.54mm:PinHeader_2x02_P2.54mm_Vertical, symbol Connector:Conn_01x04_Male
- added C? (x2): .0022u, Capacitor_SMD:C_0603_1608Metric, symbol Device:C_Small
- added C? (x2): 100uF, Capacitor_SMD:C_1210_3225Metric, symbol Device:C_Small
- added C? (x2): .0047u, Capacitor_SMD:C_0603_1608Metric, symbol Device:C_Small
- added C? (x2): 330p, Capacitor_SMD:C_0603_1608Metric, symbol Device:C_Small
- added J?: Conn_ADC, Connector_PinHeader_2.54mm:PinHeader_1x04_P2.54mm_Vertical, symbol Connector:Conn_01x04_Male
- added J?: Conn_ADC, Connector_PinHeader_2.54mm:PinHeader_2x02_P2.54mm_Vertical, symbol Connector:Conn_01x04_Male
- added J?: Conn_02x02_Odd_Even, Connector_PinHeader_2.54mm:PinHeader_2x02_P2.54mm_Vertical, symbol Connector_Generic:Conn_02x02_Odd_Even
- added R? (x2): 2.8k, Resistor_SMD:R_0603_1608Metric, symbol Device:R_Small_US
- added R? (x2): 12k, Resistor_SMD:R_0603_1608Metric, symbol Device:R_Small_US
- added R? (x2): 110k, Resistor_SMD:R_0603_1608Metric, symbol Device:R_Small_US
- added R? (x2): 36k, Resistor_SMD:R_0603_1608Metric, symbol Device:R_Small_US
- added R? (x2): 1.4k, Resistor_SMD:R_0603_1608Metric, symbol Device:R_Small_US
- added TP? (x2): LED_CTL, Connector_PinHeader_2.54mm:PinHeader_1x01_P2.54mm_Vertical, symbol Connector:TestPoint
- added TP? (x2): PWM_DAC_Out, Connector_PinHeader_2.54mm:PinHeader_1x01_P2.54mm_Vertical, symbol Connector:TestPoint
- added U? (x3): LM358, DIP08, symbol SparkFun-IC-Amplifiers:LM358
- added U?: LM7812_TO220, Package_TO_SOT_THT:TO-220-3_Vertical, symbol Regulator_Linear:LM7812_TO220
- added U?: LM7912_TO220, Package_TO_SOT_THT:TO-220-3_Vertical, symbol Regulator_Linear:LM7912_TO220
- added U?: LM358DT, digikey-footprints:SOIC-8_W3.9mm, symbol dk_Linear-Amplifiers-Instrumentation-OP-Amps-Buffer-Amps:LM358DT
Connections:
- net +15V: now also U?.3 (VO); no longer J22.3 (Pin_3)
- net -15V: now also U?.3 (VO); no longer J22.1 (Pin_1)
- net GND: now also C?.1, C?.1, C?.1, C?.2, C?.2, C?.2, J?.1 (Pin_1), J?.1 (Pin_1), J?.3 (Pin_3), J?.3 (Pin_3), R?.2, R?.2, U?.1 (GND), U?.2 (GND)
- net at J18.4 (Pin_4): now also R?.1
- net at J18.2 (Pin_2): now also R?.1
- new net: C?.1, R?.1, TP?.1, U?.1 (OUT), U?.3 (+IN)
- new net: C?.2, R?.1, R?.2 (x4)
- new net: J?.1 (Pin_1), R?.1, R?.2, TP?.1
- new net: J?.2 (Pin_2), J?.2 (Pin_2), J?.4 (Pin_4)
- new net: J?.2 (Pin_2), J?.4 (Pin_4), J?.4 (Pin_4)
- new net: C?.1, R?.1, TP?.1, U?.5 (+IN), U?.7 (OUT)
- new net: C?.1, R?.2, U?.6 (-IN)
- new net: C?.1, R?.2, U?.2 (-IN)
- new net: C?.1, J22.3 (Pin_3), U?.1 (VI)
- new net: C?.2, J22.1 (Pin_1), U?.2 (VI)
- new net: J?.3 (Pin_3), R?.1, R?.2, TP?.1
Other:
- moved on the sheet: C1, C10, C11, C12, C13, C14, C15, C16, C17, C18, C19, C2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

Commit message: Check in for Phil
Parts:
- removed C? (x2): 100uF, Capacitor_SMD:C_1210_3225Metric, symbol Device:C_Small
- removed U?: LM7812_TO220, Package_TO_SOT_THT:TO-220-3_Vertical, symbol Regulator_Linear:LM7812_TO220
- removed U?: LM7912_TO220, Package_TO_SOT_THT:TO-220-3_Vertical, symbol Regulator_Linear:LM7912_TO220
- removed U?: LM358DT, digikey-footprints:SOIC-8_W3.9mm, symbol dk_Linear-Amplifiers-Instrumentation-OP-Amps-Buffer-Amps:LM358DT
- added C28, C29, C43, C45: 100uF, Capacitor_SMD:C_1210_3225Metric, symbol Device:C_Small
- added R78, R80, R81, R84: 110k, Resistor_SMD:R_0603_1608Metric, symbol Device:R_Small_US
- added U19: LM7812_TO220, Package_TO_SOT_THT:TO-220-3_Vertical, symbol Regulator_Linear:LM7812_TO220
- added U25: LM7912_TO220, Package_TO_SOT_THT:TO-220-3_Vertical, symbol Regulator_Linear:LM7912_TO220
- J10: value (Y) -> (X)
- J9: value (X) -> (Y)
- U30: renamed from U?; footprint DIP08 -> Package_SO:SOIC-8_3.9x4.9mm_P1.27mm
- gave numbers to parts that had none: 23
Connections:
- net +15V: now also J22.3 (Pin_3), U30.8 (P$V+), C45.1, U19.1 (VI); no longer C18.1, C3.1, FB1.1
- net -15V: now also J22.1 (Pin_1), U30.4 (P$V-), C43.2, U25.2 (VI); no longer C19.2, C4.2, FB3.1
- net GND: now also C43.1, C45.2, R78.1, R80.2, R81.1, R84.2, U19.2 (GND), U25.1 (GND)
- net Pos_A(+): now also R78.2
- net Pos_A(-): now also R80.1
- net Pos_B(+): now also R81.2
- net Pos_B(-): now also R84.1
- net at C42.1, R75.1, TP10.1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: now also U30.2 (-IN); no longer U30.3 (+IN)
- net ADC (Y): now reaches J12.2 (Pin_2), J13.4 (Pin_4), J5.2 (Pin_2)
- net ADC (X): now reaches J12.4 (Pin_4), J13.2 (Pin_2), J5.4 (Pin_4)
- net at C41.1, R62.1, TP9.1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: now also U30.6 (-IN); no longer U30.5 (+IN)
- net at C35.1, R60.2: now also U30.5 (+IN); no longer U30.6 (-IN)
- net DAC (Y): now reaches J20.1 (Pin_1), J21.1 (Pin_1), J6.1 (Pin_1)
- net DAC (X): now reaches J20.3 (Pin_3), J21.3 (Pin_3), J6.3 (Pin_3)
- net at C39.1, R61.2: now also U30.3 (+IN); no longer U30.2 (-IN)
- net at FB2.1, J8.2 (Pin_2): now also C28.1, C29.2
- net at FB3.2, J8.1 (Pin_1): now also C28.2
- net at FB1.2, J8.3 (Pin_3): now also C29.1
- new net: C19.2, C4.2, FB3.1, U25.3 (VO)
- new net: C18.1, C3.1, FB1.1, U19.3 (VO)
Other:
- moved on the sheet: C18, C19, C3, C4, FB1, FB2, FB3, GalvoA_Gain1, GalvoA_Offset1, GalvoB_Gain1, GalvoB_Offset1, J1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

Commit message: More changes, added boot jumper
Parts:
- removed TP10, TP9: PWM_DAC_Out, Connector_PinHeader_2.54mm:PinHeader_1x01_P2.54mm_Vertical, symbol Connector:TestPoint
- added D6: SM4007PL, Diode_SMD:D_SOD-123F, symbol Diode:1N4007
- added J19: time_dilation, Connector_PinHeader_2.54mm:PinHeader_1x02_P2.54mm_Vertical, symbol Connector:Conn_01x02_Male
- added U26: 74LVC1G34, Package_TO_SOT_SMD:SOT-23-5, symbol project:74LVC1G34
- C1, C10, C11, C12, C13, C14, C15, C16, C17, C18, C19, C2, C20, C21, C23, C24, C26, C27, C28, C29, C3, C31, C36, C4, C40, C43, C44, C45, C47, C48, C49, C5, C50, C6, C7, C8, C9, Cam_Input1, Cam_Output1, D1, D10, D2, D3, D4, D5, D7, D9, FB1, FB2, FB3, GalvoA_Gain1, GalvoA_Offset1, GalvoB_Gain1, GalvoB_Offset1, InputA_Gain1, InputA_offset1, InputB_Gain1, InputB_offset1, K1, LED_Temp1, LED_Trigger1, Q1, R10, R11, R12, R13, R14, R15, R16, R17, R18, R19, R20, R21, R38, R39, R40, R41, R58, R59, R67, R69, R71, R78, R80, R81, R84, R9, R92, R93, S1, S2, U1, U12, U13, U14, U15, U17, U18, U2, U20, U21, U22, U28, U29, U3, U31, U32, U33, U34, U35, U4, U5, U6, U7, U8, U9: LCSL (none) -> x
- C22, C25: LCSC (none) -> C249527; LCSL C90143 -> x
- C30, C34: value .0047u -> 100pF; LCSC C159797 -> C14858; LCSL (none) -> x
- C32, C33, C37, C38: LCSC (none) -> C14858; LCSL (none) -> x
- C35: value 330p -> 10p; LCSC C1664 -> C1634; LCSL (none) -> x
- C39: value 330p -> 10pF; LCSC C1664 -> C1634; LCSL (none) -> x
- C41, C42: value .0022u -> 33pF; LCSC C33353 -> C1663; LCSL (none) -> x
- D8: LCSC (none) -> C545375; LCSL (none) -> x
- DC1, DC2: LCSC (none) -> C2286; LCSL (none) -> x
- J1: value (Y) -> (Y) FB; LCSC C124376 -> C144394; LCSL (none) -> x
- J10: value (X) -> Drive (X); LCSC C124376 -> C144394
- J11: LCSC (none) -> C124378
- J14: value Conn_POS_input_A -> POS_input_X
- J15: value Conn_POS_input_B -> POS_input_Y
- J2: value (X) -> (X) FB; LCSC C124376 -> C144394; LCSL (none) -> x
- J22: value Conn_01x03_Amp_power -> Amp_power
- J27, J3: LCSC (none) -> C124383; LCSL (none) -> x
- J29, J38, J43, J44, J45, J46, J47, J48: LCSC (none) -> C160334
- J30: LCSC (none) -> C190083
- J32, J34, J35, J36, J37: LCSC (none) -> C27543
- J39, J40, J41, J42: LCSC (none) -> C124381
- J4: LCSC C124378 -> C504991; LCSL (none) -> x
- J8: value Conn_Galvo_Power -> Galvo_Power_input; LCSC C124376 -> C29275
- J9: value (Y) -> Drive (Y); LCSC C124376 -> C144394
- R1, R2, R22, R23, R24, R25, R26, R27, R28, R29, R3, R30, R31, R32, R33, R34, R35, R36, R37, R4, R5, R6, R7, R8: LCSC (none) -> C25804; LCSL (none) -> x
- R42: value 1.4k -> 1.87k; LCSL (none) -> x
- R43: value 2.8k -> 1.07k; LCSL (none) -> x
- R44, R45, R46, R47, R56, R63: value 440 -> 442; LCSC (none) -> C23057; LCSL (none) -> x
- R48, R49, R50, R51: value 5k -> 4.7k; LCSC (none) -> C23162; LCSL (none) -> x
- R52, R74: footprint Capacitor_SMD:C_0603_1608Metric -> Resistor_SMD:R_0603_1608Metric; LCSC (none) -> C22965; LCSL (none) -> x
- R53, R72: footprint Capacitor_SMD:C_0603_1608Metric -> Resistor_SMD:R_0603_1608Metric; LCSC (none) -> C23137; LCSL (none) -> x
- R54: LCSC (none) -> C22775; LCSL (none) -> x
- R55, R57: value 12k -> 11k; LCSC C22790 -> C25950; LCSL (none) -> x
- R60, R61: value 36k -> 30k; LCSC C23147 -> C22984; LCSL (none) -> x
- R62, R75: value 1.4k -> 4.7k; LCSC C25957 -> C23162; LCSL (none) -> x
- R64: LCSC (none) -> C26096; LCSL (none) -> x
- R65: LCSC (none) -> C23178; LCSL (none) -> x
- R66, R68, R70: footprint Capacitor_SMD:C_0603_1608Metric -> Resistor_SMD:R_0603_1608Metric
- R73, R76: value 2.8k -> 4.7k; LCSC C22947 -> C23162; LCSL (none) -> x
- R77: LCSC (none) -> C25819; LCSL (none) -> x
- R79, R83, R86, R88: LCSC (none) -> C21190; LCSL (none) -> x
- R82: LCSC (none) -> C23265; LCSL (none) -> x
- TP11: value LED_CTL -> ADC_X
- TP12: value LED_CTL -> ADC_Y
- U19: LCSC (none) -> C427633; LCSL (none) -> x
- U23, U24: LCSC (none) -> C465732; LCSL (none) -> x
- U25: LCSC (none) -> C428906; LCSL (none) -> x
- U27: LCSC (none) -> C13482; LCSL (none) -> x
- U29, U30: LCSC (none) -> C9418; LCSL (none) -> x
Connections:
- net +15V: now also U19.3 (VO); no longer U19.1 (VI)
- net +5V: now also U26.5 (VCC)
- net -15V: now also U25.3 (VO); no longer U25.2 (VI)
- net GND: now also U26.1, U26.3 (GND)
- net Laser_Interlock: now also U26.2; no longer J36.2 (Pin_2), R86.2, R88.2
- net at C19.2, C4.2, FB3.1: now also U25.2 (VI); no longer U25.3 (VO)
- net at C18.1, C3.1, FB1.1: now also U19.1 (VI); no longer U19.3 (VO)
- net at J41.6 (Pin_6), U23.9 (P05): now also J19.2 (Pin_2)
- net time_dilation: now reaches U10.11 (9_OUT1C)
- net time_dilation: now also J19.1 (Pin_1)
- net at J36.1 (Pin_1), K1.2, R79.2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: now also D6.1 (K)
- net at D9.1 (K), J30.23 (P23), J34.2 (Pin_2)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: now also D6.2 (A)
- new net: J36.2 (Pin_2), R86.2, R88.2, U26.4
- no-connect marks 95 -> 94
Other:
- note added: "Bessel filter low-pass fc=60kHz Phase(1000Hz) = -1 deg Phase(10000Hz) = -9 deg"
- note added: "Power"

Commit message: R2
Parts:
- added J49: Conn_02x02_Odd_Even, Connector_PinHeader_2.54mm:PinHeader_2x02_P2.54mm_Vertical, symbol Connector_Generic:Conn_02x02_Odd_Even
- J30: footprint Connector_Dsub:DSUB-25_Female_Horizontal_P2.77x2.84mm_EdgePinOffset4.94mm_Housed_MountingHolesOffset7.48mm -> Connector_Dsub:DSUB-25_Female_Horizontal_P2.77x2.84mm_EdgePinOffset7.70mm_Housed_MountingHolesOffset9.12mm
- R66: value -- -> 1.87k; LCSC (none) -> C25957
Connections:
- net LED_PWM: now also J49.2 (Pin_2), J49.4 (Pin_4); no longer TP3.1, U12.1
- net LED_trigger_teensy: now reaches U10.3 (1_TX1_CTX2_MISO1)
- net LED_trigger_teensy: now also J49.1 (Pin_1)
- new net: J49.3 (Pin_3), TP3.1, U12.1
- no-connect marks 94 -> 93
