File: brass_board/PCB/main_board/_autosave-main_board.kicad_sch (KiCad schematic)
At the start: 133 parts

Commit message: Placement done
Parts:
- C16, C17, C18, C19, C20, C21: renamed from C?; value 100uF -> (none); footprint Capacitor_SMD:C_1210_3225Metric -> (none)
- gave numbers to parts that had none: 2
Changed lines of the file:
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@@
   (symbol (lib_id "Device:C_Small") (at 365.76 203.2 0) (unit 1)
     (in_bom yes) (on_board yes)
-    (property "Reference" "C?" (id 0) (at 369.57 201.93 0)
+    (property "Reference" "C18" (id 0) (at 369.57 201.93 0)
       (effects (font (size 1.27 1.27)) (justify left))
     )
-    (property "Value" "100uF" (id 1) (at 369.57 204.47 0)
+    (property "Value" "" (id 1) (at 369.57 204.47 0)
       (effects (font (size 1.27 1.27)) (justify left))
     )
-    (property "Footprint" "Capacitor_SMD:C_1210_3225Metric" (id 2) (at 365.76 203.2 0)
+    (property "Footprint" "" (id 2) (at 365.76 203.2 0)
       (effects (font (size 1.27 1.27)) hide)
     )
@@
   (symbol (lib_id "Device:C_Small") (at 417.83 74.93 0) (unit 1)
     (in_bom yes) (on_board yes) (fields_autoplaced)
-    (property "Reference" "C?" (id 0) (at 420.37 73.6662 0)
+    (property "Reference" "C20" (id 0) (at 420.37 73.6662 0)
       (effects (font (size 1.27 1.27)) (justify left))
     )
-    (property "Value" "100uF" (id 1) (at 420.37 76.2062 0)
+    (property "Value" "" (id 1) (at 420.37 76.2062 0)
       (effects (font (size 1.27 1.27)) (justify left))
     )
-    (property "Footprint" "Capacitor_SMD:C_1210_3225Metric" (id 2) (at 417.83 74.93 0)
+    (property "Footprint" "" (id 2) (at 417.83 74.93 0)
       (effects (font (size 1.27 1.27)) hide)
     )
@@
   (symbol (lib_id "Device:C_Small") (at 152.4 270.51 0) (unit 1)
     (in_bom yes) (on_board yes) (fields_autoplaced)
-    (property "Reference" "C?" (id 0) (at 154.94 269.2462 0)
+    (property "Reference" "C17" (id 0) (at 154.94 269.2462 0)
       (effects (font (size 1.27 1.27)) (justify left))
     )
-    (property "Value" "100uF" (id 1) (at 154.94 271.7862 0)
+    (property "Value" "" (id 1) (at 154.94 271.7862 0)
       (effects (font (size 1.27 1.27)) (justify left))
     )
-    (property "Footprint" "Capacitor_SMD:C_1210_3225Metric" (id 2) (at 152.4 270.51 0)
+    (property "Footprint" "" (id 2) (at 152.4 270.51 0)
       (effects (font (size 1.27 1.27)) hide)
     )
@@
   (symbol (lib_id "Device:C_Small") (at 152.4 261.62 0) (unit 1)
     (in_bom yes) (on_board yes) (fields_autoplaced)
-    (property "Reference" "C?" (id 0) (at 154.94 260.3562 0)
+    (property "Reference" "C16" (id 0) (at 154.94 260.3562 0)
       (effects (font (size 1.27 1.27)) (justify left))
     )
-    (property "Value" "100uF" (id 1) (at 154.94 262.8962 0)
+    (property "Value" "" (id 1) (at 154.94 262.8962 0)
       (effects (font (size 1.27 1.27)) (justify left))
     )
-    (property "Footprint" "Capacitor_SMD:C_1210_3225Metric" (id 2) (at 152.4 261.62 0)
+    (property "Footprint" "" (id 2) (at 152.4 261.62 0)
       (effects (font (size 1.27 1.27)) hide)
     )
@@
   (symbol (lib_id "Device:C_Small") (at 76.2 50.8 0) (unit 1)
     (in_bom yes) (on_board yes) (fields_autoplaced)
-    (property "Reference" "C?" (id 0) (at 78.74 49.5362 0)
+    (property "Reference" "C14" (id 0) (at 78.74 49.5362 0)
       (effects (font (size 1.27 1.27)) (justify left))
     )
@@
   (symbol (lib_id "Device:C_Small") (at 365.76 215.9 0) (unit 1)
     (in_bom yes) (on_board yes) (fields_autoplaced)
-    (property "Reference" "C?" (id 0) (at 368.3 214.6362 0)
+    (property "Reference" "C19" (id 0) (at 368.3 214.6362 0)
       (effects (font (size 1.27 1.27)) (justify left))
     )
-    (property "Value" "100uF" (id 1) (at 368.3 217.1762 0)
+    (property "Value" "" (id 1) (at 368.3 217.1762 0)
       (effects (font (size 1.27 1.27)) (justify left))
     )
-    (property "Footprint" "Capacitor_SMD:C_1210_3225Metric" (id 2) (at 365.76 215.9 0)
+    (property "Footprint" "" (id 2) (at 365.76 215.9 0)
       (effects (font (size 1.27 1.27)) hide)
     )
@@
   (symbol (lib_id "Device:C_Small") (at 114.3 50.8 0) (unit 1)
     (in_bom yes) (on_board yes) (fields_autoplaced)
-    (property "Reference" "C?" (id 0) (at 116.84 49.5362 0)
+    (property "Reference" "C15" (id 0) (at 116.84 49.5362 0)
       (effects (font (size 1.27 1.27)) (justify left))
     )
@@
   (symbol (lib_id "Device:C_Small") (at 417.83 85.09 0) (unit 1)
     (in_bom yes) (on_board yes) (fields_autoplaced)
-    (property "Reference" "C?" (id 0) (at 420.37 83.8262 0)
+    (property "Reference" "C21" (id 0) (at 420.37 83.8262 0)
       (effects (font (size 1.27 1.27)) (justify left))
     )
-    (property "Value" "100uF" (id 1) (at 420.37 86.3662 0)
+    (property "Value" "" (id 1) (at 420.37 86.3662 0)
       (effects (font (size 1.27 1.27)) (justify left))
     )
-    (property "Footprint" "Capacitor_SMD:C_1210_3225Metric" (id 2) (at 417.83 85.09 0)
+    (property "Footprint" "" (id 2) (at 417.83 85.09 0)
       (effects (font (size 1.27 1.27)) hide)
     )
@@
       (reference "C13") (unit 1) (value "C_Small") (footprint "Capacitor_SMD:C_0603_1608Metric")
     )
-    (path "/0861900d-2e75-40c6-8170-d042b0939a44"
-      (reference "C?") (unit 1) (value "100uF") (footprint "Capacitor_SMD:C_1210_3225Metric")
-    )
-    (path "/1a3765c0-2a9c-418b-8a06-dce17e04e3cd"
-      (reference "C?") (unit 1) (value "100uF") (footprint "Capacitor_SMD:C_1210_3225Metric")
+    (path "/b5c0c37c-1793-44b7-a6e1-d560bdf30c3c"
+      (reference "C14") (unit 1) (value "100uF") (footprint "Capacitor_SMD:C_1210_3225Metric")
     )
-    (path "/24b1089d-9ce7-4889-9788-0ac265ee75d3"
-      (reference "C?") (unit 1) (value "100uF") (footprint "Capacitor_SMD:C_1210_3225Metric")
+    (path "/e998cc7c-bb3d-4403-b2f4-99882c8bca86"
+      (reference "C15") (unit 1) (value "100uF") (footprint "Capacitor_SMD:C_1210_3225Metric")
     )
     (path "/b2ac8b72-8670-43fe-aafc-1e16170dc436"
-      (reference "C?") (unit 1) (value "100uF") (footprint "Capacitor_SMD:C_1210_3225Metric")
+      (reference "C16") (unit 1) (value "100uF") (footprint "Capacitor_SMD:C_1210_3225Metric")
     )
-    (path "/b5c0c37c-1793-44b7-a6e1-d560bdf30c3c"
-      (reference "C?") (unit 1) (value "100uF") (footprint "Capacitor_SMD:C_1210_3225Metric")
+    (path "/24b1089d-9ce7-4889-9788-0ac265ee75d3"
+      (reference "C17") (unit 1) (value "100uF") (footprint "Capacitor_SMD:C_1210_3225Metric")
+    )
+    (path "/0861900d-2e75-40c6-8170-d042b0939a44"
+      (reference "C18") (unit 1) (value "100uF") (footprint "Capacitor_SMD:C_1210_3225Metric")
     )
     (path "/c95a5ce1-3bae-4da1-95c8-148cb1190a6c"
-      (reference "C?") (unit 1) (value "100uF") (footprint "Capacitor_SMD:C_1210_3225Metric")
+      (reference "C19") (unit 1) (value "100uF") (footprint "Capacitor_SMD:C_1210_3225Metric")
     )
-    (path "/e998cc7c-bb3d-4403-b2f4-99882c8bca86"
-      (reference "C?") (unit 1) (value "100uF") (footprint "Capacitor_SMD:C_1210_3225Metric")
+    (path "/1a3765c0-2a9c-418b-8a06-dce17e04e3cd"
+      (reference "C20") (unit 1) (value "100uF") (footprint "Capacitor_SMD:C_1210_3225Metric")
     )
     (path "/ed307208-24a2-4c38-bd37-b69b068ac55b"
-      (reference "C?") (unit 1) (value "100uF") (footprint "Capacitor_SMD:C_1210_3225Metric")
+      (reference "C21") (unit 1) (value "100uF") (footprint "Capacitor_SMD:C_1210_3225Metric")
     )
     (path "/a4b589db-0333-4020-beb7-903028d7dbe2"
@@
     )
     (path "/b9959fab-2380-42b5-87a1-e0c1a5164d00"
-      (reference "J6") (unit 1) (value "Conn_ADC") (footprint "Connector_PinHeader_2.54mm:PinHeader_1x03_P2.54mm_Vertical")
+      (reference "J6") (unit 1) (value "Conn_DAC") (footprint "Connector_PinHeader_2.54mm:PinHeader_1x03_P2.54mm_Vertical")
     )
     (path "/389d7c04-db11-4d85-bad0-c152bf53aebe"
@@
     )
     (path "/c5cedc2a-13f9-40bc-b3c6-5d2783e59749"
-      (reference "J20") (unit 1) (value "Conn_ADC") (footprint "Connector_PinHeader_2.54mm:PinHeader_1x03_P2.54mm_Vertical")
+      (reference "J20") (unit 1) (value "Conn_DAC") (footprint "Connector_PinHeader_2.54mm:PinHeader_1x03_P2.54mm_Vertical")
     )
     (path "/3a5c058e-5bc1-4fb4-a6fe-0b902857168c"
@@
     )
     (path "/4bed2ed8-4f7e-4663-ad51-f71d004dc427"
-      (reference "U11") (unit 1) (value "Teensy4.0") (footprint "teensy:Teensy30_31_32_All_Pins")
+      (reference "U11") (unit 1) (value "Teensy4.0") (footprint "teensy:Teensy40")
     )
     (path "/5373c0be-ff3a-4547-9cf1-d7df2fb62b87"
